File: Kicad/8086testCircuit.kicad_pcb (KiCad board)
At the start: 2 copper layers, 11 parts, among them SW1 RST, U1 8086_Min_Mode, U10 74HCT573, U11 74HCT245, U2 8284, U4 74HCT138, U7 74HCT573, U8 74HCT245, U9 74HCT573, Y1 Crystal 30MHz

Commit message: Add files via upload
Parts:
- U1: value 8086_Min_Mode -> 8086-1_Min_Mode
Connections:
- U1 pad 17: unconnected-(U1-NMI-Pad17) -> /CPU/NMI
- U1 pad 18: unconnected-(U1-INTR-Pad18) -> /CPU/INTR
- U1 pad 23: unconnected-(U1-~{TEST}-Pad23) -> /CPU/!TEST
- U1 pad 24: unconnected-(U1-~{INTA}-Pad24) -> /CPU/!INTA
- U1 pad 30: unconnected-(U1-HLDA-Pad30) -> /CPU/HLDA
- U1 pad 31: unconnected-(U1-HOLD-Pad31) -> /CPU/HOLD
- U1 pad 33: unconnected-(U1-MN/~{MX}-Pad33) -> /CPU/5V
- U10 pad 15: unconnected-(U10-Q4-Pad15) -> /CPU/!BHE
- U10 pad 16: unconnected-(U10-Q3-Pad16) -> /CPU/ADDR19
- U10 pad 17: unconnected-(U10-Q2-Pad17) -> /CPU/ADDR18
- U10 pad 18: unconnected-(U10-Q1-Pad18) -> /CPU/ADDR17
- U10 pad 19: unconnected-(U10-Q0-Pad19) -> /CPU/ADDR16
- U11 pad 11: unconnected-(U11-B7-Pad11) -> /CPU/DATA15
- U11 pad 12: unconnected-(U11-B6-Pad12) -> /CPU/DATA14
- U11 pad 13: unconnected-(U11-B5-Pad13) -> /CPU/DATA13
- U11 pad 14: unconnected-(U11-B4-Pad14) -> /CPU/DATA12
- U11 pad 15: unconnected-(U11-B3-Pad15) -> /CPU/DATA11
- U11 pad 16: unconnected-(U11-B2-Pad16) -> /CPU/DATA10
- U11 pad 17: unconnected-(U11-B1-Pad17) -> /CPU/DATA9
- U11 pad 18: unconnected-(U11-B0-Pad18) -> /CPU/DATA8
- U7 pad 12: unconnected-(U7-Q7-Pad12) -> /CPU/ADDR7
- U7 pad 13: unconnected-(U7-Q6-Pad13) -> /CPU/ADDR6
- U7 pad 14: unconnected-(U7-Q5-Pad14) -> /CPU/ADDR5
- U7 pad 15: unconnected-(U7-Q4-Pad15) -> /CPU/ADDR4
- U7 pad 16: unconnected-(U7-Q3-Pad16) -> /CPU/ADDR3
- U7 pad 17: unconnected-(U7-Q2-Pad17) -> /CPU/ADDR2
- U7 pad 18: unconnected-(U7-Q1-Pad18) -> /CPU/ADDR1
- U7 pad 19: unconnected-(U7-Q0-Pad19) -> /CPU/ADDR0
- U8 pad 11: unconnected-(U8-B7-Pad11) -> /CPU/DATA7
- U8 pad 12: unconnected-(U8-B6-Pad12) -> /CPU/DATA6
- U8 pad 13: unconnected-(U8-B5-Pad13) -> /CPU/DATA5
- U8 pad 14: unconnected-(U8-B4-Pad14) -> /CPU/DATA4
- U8 pad 15: unconnected-(U8-B3-Pad15) -> /CPU/DATA3
- U8 pad 16: unconnected-(U8-B2-Pad16) -> /CPU/DATA2
- U8 pad 17: unconnected-(U8-B1-Pad17) -> /CPU/DATA1
- U8 pad 18: unconnected-(U8-B0-Pad18) -> /CPU/DATA0
- U9 pad 12: unconnected-(U9-Q7-Pad12) -> /CPU/ADDR15
- U9 pad 13: unconnected-(U9-Q6-Pad13) -> /CPU/ADDR14
- U9 pad 14: unconnected-(U9-Q5-Pad14) -> /CPU/ADDR13
- U9 pad 15: unconnected-(U9-Q4-Pad15) -> /CPU/ADDR12
- U9 pad 16: unconnected-(U9-Q3-Pad16) -> /CPU/ADDR11
- U9 pad 17: unconnected-(U9-Q2-Pad17) -> /CPU/ADDR10
- U9 pad 18: unconnected-(U9-Q1-Pad18) -> /CPU/ADDR9
- U9 pad 19: unconnected-(U9-Q0-Pad19) -> /CPU/ADDR8
Changed lines of the file:
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@@
 			(layers "*.Cu" "*.Mask")
 			(remove_unused_layers no)
-			(net "unconnected-(U10-Q4-Pad15)")
+			(net "/CPU/!BHE")
 			(pinfunction "Q4_15")
 			(pintype "tri_state")
@@
 			(layers "*.Cu" "*.Mask")
 			(remove_unused_layers no)
-			(net "unconnected-(U10-Q3-Pad16)")
+			(net "/CPU/ADDR19")
 			(pinfunction "Q3_16")
 			(pintype "tri_state")
@@
 			(layers "*.Cu" "*.Mask")
 			(remove_unused_layers no)
-			(net "unconnected-(U10-Q2-Pad17)")
+			(net "/CPU/ADDR18")
 			(pinfunction "Q2_17")
 			(pintype "tri_state")
@@
 			(layers "*.Cu" "*.Mask")
 			(remove_unused_layers no)
-			(net "unconnected-(U10-Q1-Pad18)")
+			(net "/CPU/ADDR17")
 			(pinfunction "Q1_18")
 			(pintype "tri_state")
@@
 			(layers "*.Cu" "*.Mask")
 			(remove_unused_layers no)
-			(net "unconnected-(U10-Q0-Pad19)")
+			(net "/CPU/ADDR16")
 			(pinfunction "Q0_19")
 			(pintype "tri_state")
@@
 			(layers "*.Cu" "*.Mask")
 			(remove_unused_layers no)
-			(net "unconnected-(U9-Q7-Pad12)")
+			(net "/CPU/ADDR15")
 			(pinfunction "Q7_12")
 			(pintype "tri_state")
@@
 			(layers "*.Cu" "*.Mask")
 			(remove_unused_layers no)
-			(net "unconnected-(U9-Q6-Pad13)")
+			(net "/CPU/ADDR14")
 			(pinfunction "Q6_13")
 			(pintype "tri_state")
@@
 			(layers "*.Cu" "*.Mask")
 			(remove_unused_layers no)
-			(net "unconnected-(U9-Q5-Pad14)")
+			(net "/CPU/ADDR13")
 			(pinfunction "Q5_14")
 			(pintype "tri_state")
@@
 			(layers "*.Cu" "*.Mask")
 			(remove_unused_layers no)
-			(net "unconnected-(U9-Q4-Pad15)")
+			(net "/CPU/ADDR12")
 			(pinfunction "Q4_15")
 			(pintype "tri_state")
@@
 			(layers "*.Cu" "*.Mask")
 			(remove_unused_layers no)
-			(net "unconnected-(U9-Q3-Pad16)")
+			(net "/CPU/ADDR11")
 			(pinfunction "Q3_16")
 			(pintype "tri_state")
@@
 			(layers "*.Cu" "*.Mask")
 			(remove_unused_layers no)
-			(net "unconnected-(U9-Q2-Pad17)")
+			(net "/CPU/ADDR10")
 			(pinfunction "Q2_17")
 			(pintype "tri_state")
@@
 			(layers "*.Cu" "*.Mask")
 			(remove_unused_layers no)
-			(net "unconnected-(U9-Q1-Pad18)")
+			(net "/CPU/ADDR9")
 			(pinfunction "Q1_18")
 			(pintype "tri_state")
@@
 			(layers "*.Cu" "*.Mask")
 			(remove_unused_layers no)
-			(net "unconnected-(U9-Q0-Pad19)")
+			(net "/CPU/ADDR8")
 			(pinfunction "Q0_19")
 			(pintype "tri_state")
@@
 			)
 		)
-		(property "Value" "8086_Min_Mode"
+		(property "Value" "8086-1_Min_Mode"
 			(at 7.62 50.59 0)
 			(layer "F.Fab")
@@
 			(layers "*.Cu" "*.Mask")
 			(remove_unused_layers no)
-			(net "unconnected-(U1-NMI-Pad17)")
+			(net "/CPU/NMI")
 			(pinfunction "NMI_17")
 			(pintype "input")
@@
 			(layers "*.Cu" "*.Mask")
 			(remove_unused_layers no)
-			(net "unconnected-(U1-INTR-Pad18)")
+			(net "/CPU/INTR")
 			(pinfunction "INTR_18")
 			(pintype "input")
@@
 			(layers "*.Cu" "*.Mask")
 			(remove_unused_layers no)
-			(net "unconnected-(U1-~{TEST}-Pad23)")
+			(net "/CPU/!TEST")
 			(pinfunction "~{TEST}_23")
 			(pintype "input")
@@
 			(layers "*.Cu" "*.Mask")
 			(remove_unused_layers no)
-			(net "unconnected-(U1-~{INTA}-Pad24)")
+			(net "/CPU/!INTA")
 			(pinfunction "~{INTA}_24")
 			(pintype "output")
@@
 			(layers "*.Cu" "*.Mask")
 			(remove_unused_layers no)
-			(net "unconnected-(U1-HLDA-Pad30)")
+			(net "/CPU/HLDA")
 			(pinfunction "HLDA_30")
 			(pintype "output")
@@
 			(layers "*.Cu" "*.Mask")
 			(remove_unused_layers no)
-			(net "unconnected-(U1-HOLD-Pad31)")
+			(net "/CPU/HOLD")
 			(pinfunction "HOLD_31")
 			(pintype "input")
@@
 			(layers "*.Cu" "*.Mask")
 			(remove_unused_layers no)
-			(net "unconnected-(U1-MN{slash}~{MX}-Pad33)")
+			(net "/CPU/5V")
 			(pinfunction "MN/~{MX}_33")
 			(pintype "input")
@@
 			(layers "*.Cu" "*.Mask")
 			(remove_unused_layers no)
-			(net "unconnected-(U7-Q7-Pad12)")
+			(net "/CPU/ADDR7")
 			(pinfunction "Q7_12")
 			(pintype "tri_state")
@@
 			(layers "*.Cu" "*.Mask")
 			(remove_unused_layers no)
-			(net "unconnected-(U7-Q6-Pad13)")
+			(net "/CPU/ADDR6")
 			(pinfunction "Q6_13")
 			(pintype "tri_state")
@@
 			(layers "*.Cu" "*.Mask")
 			(remove_unused_layers no)
-			(net "unconnected-(U7-Q5-Pad14)")
+			(net "/CPU/ADDR5")
 			(pinfunction "Q5_14")
 			(pintype "tri_state")
@@
 			(layers "*.Cu" "*.Mask")
 			(remove_unused_layers no)
-			(net "unconnected-(U7-Q4-Pad15)")
+			(net "/CPU/ADDR4")
 			(pinfunction "Q4_15")
 			(pintype "tri_state")
@@
 			(layers "*.Cu" "*.Mask")
 			(remove_unused_layers no)
-			(net "unconnected-(U7-Q3-Pad16)")
+			(net "/CPU/ADDR3")
 			(pinfunction "Q3_16")
 			(pintype "tri_state")
@@
 			(layers "*.Cu" "*.Mask")
 			(remove_unused_layers no)
-			(net "unconnected-(U7-Q2-Pad17)")
+			(net "/CPU/ADDR2")
 			(pinfunction "Q2_17")
 			(pintype "tri_state")
@@
 			(layers "*.Cu" "*.Mask")
 			(remove_unused_layers no)
-			(net "unconnected-(U7-Q1-Pad18)")
+			(net "/CPU/ADDR1")
 			(pinfunction "Q1_18")
 			(pintype "tri_state")
@@
 			(layers "*.Cu" "*.Mask")
 			(remove_unused_layers no)
-			(net "unconnected-(U7-Q0-Pad19)")
+			(net "/CPU/ADDR0")
 			(pinfunction "Q0_19")
 			(pintype "tri_state")
@@
 			(layers "*.Cu" "*.Mask")
 			(remove_unused_layers no)
-			(net "unconnected-(U8-B7-Pad11)")
+			(net "/CPU/DATA7")
 			(pinfunction "B7_11")
 			(pintype "tri_state")
@@
 			(layers "*.Cu" "*.Mask")
 			(remove_unused_layers no)
-			(net "unconnected-(U8-B6-Pad12)")
+			(net "/CPU/DATA6")
 			(pinfunction "B6_12")
 			(pintype "tri_state")
@@
 			(layers "*.Cu" "*.Mask")
 			(remove_unused_layers no)
-			(net "unconnected-(U8-B5-Pad13)")
+			(net "/CPU/DATA5")
 			(pinfunction "B5_13")
 			(pintype "tri_state")
@@
 			(layers "*.Cu" "*.Mask")
 			(remove_unused_layers no)
-			(net "unconnected-(U8-B4-Pad14)")
+			(net "/CPU/DATA4")
 			(pinfunction "B4_14")
 			(pintype "tri_state")
@@
 			(layers "*.Cu" "*.Mask")
 			(remove_unused_layers no)
-			(net "unconnected-(U8-B3-Pad15)")
+			(net "/CPU/DATA3")
 			(pinfunction "B3_15")
 			(pintype "tri_state")
@@
 			(layers "*.Cu" "*.Mask")
 			(remove_unused_layers no)
-			(net "unconnected-(U8-B2-Pad16)")
+			(net "/CPU/DATA2")
 			(pinfunction "B2_16")
 			(pintype "tri_state")
@@
 			(layers "*.Cu" "*.Mask")
 			(remove_unused_layers no)
-			(net "unconnected-(U8-B1-Pad17)")
+			(net "/CPU/DATA1")
 			(pinfunction "B1_17")
 			(pintype "tri_state")
@@
 			(layers "*.Cu" "*.Mask")
 			(remove_unused_layers no)
-			(net "unconnected-(U8-B0-Pad18)")
+			(net "/CPU/DATA0")
 			(pinfunction "B0_18")
 			(pintype "tri_state")
@@
 			(layers "*.Cu" "*.Mask")
 			(remove_unused_layers no)
-			(net "unconnected-(U11-B7-Pad11)")
+			(net "/CPU/DATA15")
 			(pinfunction "B7_11")
 			(pintype "tri_state")
@@
 			(layers "*.Cu" "*.Mask")
 			(remove_unused_layers no)
-			(net "unconnected-(U11-B6-Pad12)")
+			(net "/CPU/DATA14")
 			(pinfunction "B6_12")
 			(pintype "tri_state")
@@
 			(layers "*.Cu" "*.Mask")
 			(remove_unused_layers no)
-			(net "unconnected-(U11-B5-Pad13)")
+			(net "/CPU/DATA13")
 			(pinfunction "B5_13")
 			(pintype "tri_state")
@@
 			(layers "*.Cu" "*.Mask")
 			(remove_unused_layers no)
-			(net "unconnected-(U11-B4-Pad14)")
+			(net "/CPU/DATA12")
 			(pinfunction "B4_14")
 			(pintype "tri_state")
@@
 			(layers "*.Cu" "*.Mask")
 			(remove_unused_layers no)
-			(net "unconnected-(U11-B3-Pad15)")
+			(net "/CPU/DATA11")
 			(pinfunction "B3_15")
 			(pintype "tri_state")
@@
 			(layers "*.Cu" "*.Mask")
 			(remove_unused_layers no)
-			(net "unconnected-(U11-B2-Pad16)")
+			(net "/CPU/DATA10")
 			(pinfunction "B2_16")
 			(pintype "tri_state")
@@
 			(layers "*.Cu" "*.Mask")
 			(remove_unused_layers no)
-			(net "unconnected-(U11-B1-Pad17)")
+			(net "/CPU/DATA9")
 			(pinfunction "B1_17")
 			(pintype "tri_state")
@@
 			(layers "*.Cu" "*.Mask")
 			(remove_unused_layers no)
-			(net "unconnected-(U11-B0-Pad18)")
+			(net "/CPU/DATA8")
 			(pinfunction "B0_18")
 			(pintype "tri_state")
