File: Kicad/8086testCircuit.kicad_sch (KiCad schematic)
At the start: 0 parts

Commit message: Add files via upload
Parts:
- added #J1: Bus_ISA_8bit_refrence, symbol Connector:Bus_ISA_8bit
- added BASICMEMORY, CLOCK, CPU, J10, J2, J6, J7, J8, J9: Conn_02x31_Row_Letter_First, Connector_PinHeader_2.54mm:PinHeader_2x31_P2.54mm_Vertical, symbol Connector_Generic:Conn_02x31_Row_Letter_First
- added J1: Conn_02x31_Row_Letter_First, symbol Connector_Generic:Conn_02x31_Row_Letter_First
Connections:
- new net: BASICMEMORY.a1 (Pin_a1), CLOCK.a1 (Pin_a1), CPU.a1 (Pin_a1), J10.a1 (Pin_a1), J6.a1 (Pin_a1), J7.a1 (Pin_a1), J8.a1 (Pin_a1), J9.a1 (Pin_a1)
- new net: BASICMEMORY.a10 (Pin_a10), CLOCK.a10 (Pin_a10), CPU.a10 (Pin_a10), J10.a10 (Pin_a10), J6.a10 (Pin_a10), J7.a10 (Pin_a10), J8.a10 (Pin_a10), J9.a10 (Pin_a10)
- new net: BASICMEMORY.a11 (Pin_a11), CLOCK.a11 (Pin_a11), CPU.a11 (Pin_a11), J10.a11 (Pin_a11), J6.a11 (Pin_a11), J7.a11 (Pin_a11), J8.a11 (Pin_a11), J9.a11 (Pin_a11)
- new net: BASICMEMORY.a12 (Pin_a12), CLOCK.a12 (Pin_a12), CPU.a12 (Pin_a12), J10.a12 (Pin_a12), J6.a12 (Pin_a12), J7.a12 (Pin_a12), J8.a12 (Pin_a12), J9.a12 (Pin_a12)
- new net: BASICMEMORY.a13 (Pin_a13), CLOCK.a13 (Pin_a13), CPU.a13 (Pin_a13), J10.a13 (Pin_a13), J6.a13 (Pin_a13), J7.a13 (Pin_a13), J8.a13 (Pin_a13), J9.a13 (Pin_a13)
- new net: BASICMEMORY.a14 (Pin_a14), CLOCK.a14 (Pin_a14), CPU.a14 (Pin_a14), J10.a14 (Pin_a14), J6.a14 (Pin_a14), J7.a14 (Pin_a14), J8.a14 (Pin_a14), J9.a14 (Pin_a14)
- new net: BASICMEMORY.a15 (Pin_a15), CLOCK.a15 (Pin_a15), CPU.a15 (Pin_a15), J10.a15 (Pin_a15), J6.a15 (Pin_a15), J7.a15 (Pin_a15), J8.a15 (Pin_a15), J9.a15 (Pin_a15)
- new net: BASICMEMORY.a16 (Pin_a16), CLOCK.a16 (Pin_a16), CPU.a16 (Pin_a16), J10.a16 (Pin_a16), J6.a16 (Pin_a16), J7.a16 (Pin_a16), J8.a16 (Pin_a16), J9.a16 (Pin_a16)
- new net: BASICMEMORY.a17 (Pin_a17), CLOCK.a17 (Pin_a17), CPU.a17 (Pin_a17), J10.a17 (Pin_a17), J6.a17 (Pin_a17), J7.a17 (Pin_a17), J8.a17 (Pin_a17), J9.a17 (Pin_a17)
- new net: BASICMEMORY.a18 (Pin_a18), CLOCK.a18 (Pin_a18), CPU.a18 (Pin_a18), J10.a18 (Pin_a18), J6.a18 (Pin_a18), J7.a18 (Pin_a18), J8.a18 (Pin_a18), J9.a18 (Pin_a18)
- new net: BASICMEMORY.a19 (Pin_a19), CLOCK.a19 (Pin_a19), CPU.a19 (Pin_a19), J10.a19 (Pin_a19), J6.a19 (Pin_a19), J7.a19 (Pin_a19), J8.a19 (Pin_a19), J9.a19 (Pin_a19)
- new net: BASICMEMORY.a2 (Pin_a2), CLOCK.a2 (Pin_a2), CPU.a2 (Pin_a2), J10.a2 (Pin_a2), J6.a2 (Pin_a2), J7.a2 (Pin_a2), J8.a2 (Pin_a2), J9.a2 (Pin_a2)
- new net: BASICMEMORY.a20 (Pin_a20), CLOCK.a20 (Pin_a20), CPU.a20 (Pin_a20), J10.a20 (Pin_a20), J6.a20 (Pin_a20), J7.a20 (Pin_a20), J8.a20 (Pin_a20), J9.a20 (Pin_a20)
- new net: BASICMEMORY.a21 (Pin_a21), CLOCK.a21 (Pin_a21), CPU.a21 (Pin_a21), J10.a21 (Pin_a21), J6.a21 (Pin_a21), J7.a21 (Pin_a21), J8.a21 (Pin_a21), J9.a21 (Pin_a21)
- new net: BASICMEMORY.a22 (Pin_a22), CLOCK.a22 (Pin_a22), CPU.a22 (Pin_a22), J10.a22 (Pin_a22), J6.a22 (Pin_a22), J7.a22 (Pin_a22), J8.a22 (Pin_a22), J9.a22 (Pin_a22)
- new net: BASICMEMORY.a23 (Pin_a23), CLOCK.a23 (Pin_a23), CPU.a23 (Pin_a23), J10.a23 (Pin_a23), J6.a23 (Pin_a23), J7.a23 (Pin_a23), J8.a23 (Pin_a23), J9.a23 (Pin_a23)
- new net: BASICMEMORY.a24 (Pin_a24), CLOCK.a24 (Pin_a24), CPU.a24 (Pin_a24), J10.a24 (Pin_a24), J6.a24 (Pin_a24), J7.a24 (Pin_a24), J8.a24 (Pin_a24), J9.a24 (Pin_a24)
- new net: BASICMEMORY.a25 (Pin_a25), CLOCK.a25 (Pin_a25), CPU.a25 (Pin_a25), J10.a25 (Pin_a25), J6.a25 (Pin_a25), J7.a25 (Pin_a25), J8.a25 (Pin_a25), J9.a25 (Pin_a25)
- new net: BASICMEMORY.a26 (Pin_a26), CLOCK.a26 (Pin_a26), CPU.a26 (Pin_a26), J10.a26 (Pin_a26), J6.a26 (Pin_a26), J7.a26 (Pin_a26), J8.a26 (Pin_a26), J9.a26 (Pin_a26)
- new net: BASICMEMORY.a27 (Pin_a27), CLOCK.a27 (Pin_a27), CPU.a27 (Pin_a27), J10.a27 (Pin_a27), J6.a27 (Pin_a27), J7.a27 (Pin_a27), J8.a27 (Pin_a27), J9.a27 (Pin_a27)
- new net: BASICMEMORY.a28 (Pin_a28), CLOCK.a28 (Pin_a28), CPU.a28 (Pin_a28), J10.a28 (Pin_a28), J6.a28 (Pin_a28), J7.a28 (Pin_a28), J8.a28 (Pin_a28), J9.a28 (Pin_a28)
- new net: BASICMEMORY.a29 (Pin_a29), CLOCK.a29 (Pin_a29), CPU.a29 (Pin_a29), J10.a29 (Pin_a29), J6.a29 (Pin_a29), J7.a29 (Pin_a29), J8.a29 (Pin_a29), J9.a29 (Pin_a29)
- new net: BASICMEMORY.a3 (Pin_a3), CLOCK.a3 (Pin_a3), CPU.a3 (Pin_a3), J10.a3 (Pin_a3), J6.a3 (Pin_a3), J7.a3 (Pin_a3), J8.a3 (Pin_a3), J9.a3 (Pin_a3)
- new net: BASICMEMORY.a30 (Pin_a30), CLOCK.a30 (Pin_a30), CPU.a30 (Pin_a30), J10.a30 (Pin_a30), J6.a30 (Pin_a30), J7.a30 (Pin_a30), J8.a30 (Pin_a30), J9.a30 (Pin_a30)
- new net: BASICMEMORY.a31 (Pin_a31), CLOCK.a31 (Pin_a31), CPU.a31 (Pin_a31), J10.a31 (Pin_a31), J6.a31 (Pin_a31), J7.a31 (Pin_a31), J8.a31 (Pin_a31), J9.a31 (Pin_a31)
- new net: BASICMEMORY.a4 (Pin_a4), CLOCK.a4 (Pin_a4), CPU.a4 (Pin_a4), J10.a4 (Pin_a4), J6.a4 (Pin_a4), J7.a4 (Pin_a4), J8.a4 (Pin_a4), J9.a4 (Pin_a4)
- new net: BASICMEMORY.a5 (Pin_a5), CLOCK.a5 (Pin_a5), CPU.a5 (Pin_a5), J10.a5 (Pin_a5), J6.a5 (Pin_a5), J7.a5 (Pin_a5), J8.a5 (Pin_a5), J9.a5 (Pin_a5)
- new net: BASICMEMORY.a6 (Pin_a6), CLOCK.a6 (Pin_a6), CPU.a6 (Pin_a6), J10.a6 (Pin_a6), J6.a6 (Pin_a6), J7.a6 (Pin_a6), J8.a6 (Pin_a6), J9.a6 (Pin_a6)
- new net: BASICMEMORY.a7 (Pin_a7), CLOCK.a7 (Pin_a7), CPU.a7 (Pin_a7), J10.a7 (Pin_a7), J6.a7 (Pin_a7), J7.a7 (Pin_a7), J8.a7 (Pin_a7), J9.a7 (Pin_a7)
- new net: BASICMEMORY.a8 (Pin_a8), CLOCK.a8 (Pin_a8), CPU.a8 (Pin_a8), J10.a8 (Pin_a8), J6.a8 (Pin_a8), J7.a8 (Pin_a8), J8.a8 (Pin_a8), J9.a8 (Pin_a8)
- new net: BASICMEMORY.a9 (Pin_a9), CLOCK.a9 (Pin_a9), CPU.a9 (Pin_a9), J10.a9 (Pin_a9), J6.a9 (Pin_a9), J7.a9 (Pin_a9), J8.a9 (Pin_a9), J9.a9 (Pin_a9)
- new net: BASICMEMORY.b1 (Pin_b1), CLOCK.b1 (Pin_b1), CPU.b1 (Pin_b1), J10.b1 (Pin_b1), J6.b1 (Pin_b1), J7.b1 (Pin_b1), J8.b1 (Pin_b1), J9.b1 (Pin_b1)
- new net: BASICMEMORY.b10 (Pin_b10), CLOCK.b10 (Pin_b10), CPU.b10 (Pin_b10), J10.b10 (Pin_b10), J6.b10 (Pin_b10), J7.b10 (Pin_b10), J8.b10 (Pin_b10), J9.b10 (Pin_b10)
- new net: BASICMEMORY.b11 (Pin_b11), CLOCK.b11 (Pin_b11), CPU.b11 (Pin_b11), J10.b11 (Pin_b11), J6.b11 (Pin_b11), J7.b11 (Pin_b11), J8.b11 (Pin_b11), J9.b11 (Pin_b11)
- new net: BASICMEMORY.b12 (Pin_b12), CLOCK.b12 (Pin_b12), CPU.b12 (Pin_b12), J10.b12 (Pin_b12), J6.b12 (Pin_b12), J7.b12 (Pin_b12), J8.b12 (Pin_b12), J9.b12 (Pin_b12)
- new net: BASICMEMORY.b13 (Pin_b13), CLOCK.b13 (Pin_b13), CPU.b13 (Pin_b13), J10.b13 (Pin_b13), J6.b13 (Pin_b13), J7.b13 (Pin_b13), J8.b13 (Pin_b13), J9.b13 (Pin_b13)
- new net: BASICMEMORY.b14 (Pin_b14), CLOCK.b14 (Pin_b14), CPU.b14 (Pin_b14), J10.b14 (Pin_b14), J6.b14 (Pin_b14), J7.b14 (Pin_b14), J8.b14 (Pin_b14), J9.b14 (Pin_b14)
- new net: BASICMEMORY.b15 (Pin_b15), CLOCK.b15 (Pin_b15), CPU.b15 (Pin_b15), J10.b15 (Pin_b15), J6.b15 (Pin_b15), J7.b15 (Pin_b15), J8.b15 (Pin_b15), J9.b15 (Pin_b15)
- new net: BASICMEMORY.b16 (Pin_b16), CLOCK.b16 (Pin_b16), CPU.b16 (Pin_b16), J10.b16 (Pin_b16), J6.b16 (Pin_b16), J7.b16 (Pin_b16), J8.b16 (Pin_b16), J9.b16 (Pin_b16)
- new net: BASICMEMORY.b17 (Pin_b17), CLOCK.b17 (Pin_b17), CPU.b17 (Pin_b17), J10.b17 (Pin_b17), J6.b17 (Pin_b17), J7.b17 (Pin_b17), J8.b17 (Pin_b17), J9.b17 (Pin_b17)
- new net: BASICMEMORY.b18 (Pin_b18), CLOCK.b18 (Pin_b18), CPU.b18 (Pin_b18), J10.b18 (Pin_b18), J6.b18 (Pin_b18), J7.b18 (Pin_b18), J8.b18 (Pin_b18), J9.b18 (Pin_b18)
- new net: BASICMEMORY.b19 (Pin_b19), CLOCK.b19 (Pin_b19), CPU.b19 (Pin_b19), J10.b19 (Pin_b19), J6.b19 (Pin_b19), J7.b19 (Pin_b19), J8.b19 (Pin_b19), J9.b19 (Pin_b19)
- new net: BASICMEMORY.b2 (Pin_b2), CLOCK.b2 (Pin_b2), CPU.b2 (Pin_b2), J10.b2 (Pin_b2), J6.b2 (Pin_b2), J7.b2 (Pin_b2), J8.b2 (Pin_b2), J9.b2 (Pin_b2)
- new net: BASICMEMORY.b20 (Pin_b20), CLOCK.b20 (Pin_b20), CPU.b20 (Pin_b20), J10.b20 (Pin_b20), J6.b20 (Pin_b20), J7.b20 (Pin_b20), J8.b20 (Pin_b20), J9.b20 (Pin_b20)
- new net: BASICMEMORY.b21 (Pin_b21), CLOCK.b21 (Pin_b21), CPU.b21 (Pin_b21), J10.b21 (Pin_b21), J6.b21 (Pin_b21), J7.b21 (Pin_b21), J8.b21 (Pin_b21), J9.b21 (Pin_b21)
- new net: BASICMEMORY.b22 (Pin_b22), CLOCK.b22 (Pin_b22), CPU.b22 (Pin_b22), J10.b22 (Pin_b22), J6.b22 (Pin_b22), J7.b22 (Pin_b22), J8.b22 (Pin_b22), J9.b22 (Pin_b22)
- new net: BASICMEMORY.b23 (Pin_b23), CLOCK.b23 (Pin_b23), CPU.b23 (Pin_b23), J10.b23 (Pin_b23), J6.b23 (Pin_b23), J7.b23 (Pin_b23), J8.b23 (Pin_b23), J9.b23 (Pin_b23)
- new net: BASICMEMORY.b24 (Pin_b24), CLOCK.b24 (Pin_b24), CPU.b24 (Pin_b24), J10.b24 (Pin_b24), J6.b24 (Pin_b24), J7.b24 (Pin_b24), J8.b24 (Pin_b24), J9.b24 (Pin_b24)
- new net: BASICMEMORY.b25 (Pin_b25), CLOCK.b25 (Pin_b25), CPU.b25 (Pin_b25), J10.b25 (Pin_b25), J6.b25 (Pin_b25), J7.b25 (Pin_b25), J8.b25 (Pin_b25), J9.b25 (Pin_b25)
- new net: BASICMEMORY.b26 (Pin_b26), CLOCK.b26 (Pin_b26), CPU.b26 (Pin_b26), J10.b26 (Pin_b26), J6.b26 (Pin_b26), J7.b26 (Pin_b26), J8.b26 (Pin_b26), J9.b26 (Pin_b26)
- new net: BASICMEMORY.b27 (Pin_b27), CLOCK.b27 (Pin_b27), CPU.b27 (Pin_b27), J10.b27 (Pin_b27), J6.b27 (Pin_b27), J7.b27 (Pin_b27), J8.b27 (Pin_b27), J9.b27 (Pin_b27)
- new net: BASICMEMORY.b28 (Pin_b28), CLOCK.b28 (Pin_b28), CPU.b28 (Pin_b28), J10.b28 (Pin_b28), J6.b28 (Pin_b28), J7.b28 (Pin_b28), J8.b28 (Pin_b28), J9.b28 (Pin_b28)
- new net: BASICMEMORY.b29 (Pin_b29), CLOCK.b29 (Pin_b29), CPU.b29 (Pin_b29), J10.b29 (Pin_b29), J6.b29 (Pin_b29), J7.b29 (Pin_b29), J8.b29 (Pin_b29), J9.b29 (Pin_b29)
- new net: BASICMEMORY.b3 (Pin_b3), CLOCK.b3 (Pin_b3), CPU.b3 (Pin_b3), J10.b3 (Pin_b3), J6.b3 (Pin_b3), J7.b3 (Pin_b3), J8.b3 (Pin_b3), J9.b3 (Pin_b3)
- new net: BASICMEMORY.b30 (Pin_b30), CLOCK.b30 (Pin_b30), CPU.b30 (Pin_b30), J10.b30 (Pin_b30), J6.b30 (Pin_b30), J7.b30 (Pin_b30), J8.b30 (Pin_b30), J9.b30 (Pin_b30)
- new net: BASICMEMORY.b31 (Pin_b31), CLOCK.b31 (Pin_b31), CPU.b31 (Pin_b31), J10.b31 (Pin_b31), J6.b31 (Pin_b31), J7.b31 (Pin_b31), J8.b31 (Pin_b31), J9.b31 (Pin_b31)
- new net: BASICMEMORY.b4 (Pin_b4), CLOCK.b4 (Pin_b4), CPU.b4 (Pin_b4), J10.b4 (Pin_b4), J6.b4 (Pin_b4), J7.b4 (Pin_b4), J8.b4 (Pin_b4), J9.b4 (Pin_b4)
- new net: BASICMEMORY.b5 (Pin_b5), CLOCK.b5 (Pin_b5), CPU.b5 (Pin_b5), J10.b5 (Pin_b5), J6.b5 (Pin_b5), J7.b5 (Pin_b5), J8.b5 (Pin_b5), J9.b5 (Pin_b5)
- new net: BASICMEMORY.b6 (Pin_b6), CLOCK.b6 (Pin_b6), CPU.b6 (Pin_b6), J10.b6 (Pin_b6), J6.b6 (Pin_b6), J7.b6 (Pin_b6), J8.b6 (Pin_b6), J9.b6 (Pin_b6)
- new net: BASICMEMORY.b7 (Pin_b7), CLOCK.b7 (Pin_b7), CPU.b7 (Pin_b7), J10.b7 (Pin_b7), J6.b7 (Pin_b7), J7.b7 (Pin_b7), J8.b7 (Pin_b7), J9.b7 (Pin_b7)
- new net: BASICMEMORY.b8 (Pin_b8), CLOCK.b8 (Pin_b8), CPU.b8 (Pin_b8), J10.b8 (Pin_b8), J6.b8 (Pin_b8), J7.b8 (Pin_b8), J8.b8 (Pin_b8), J9.b8 (Pin_b8)
- new net: BASICMEMORY.b9 (Pin_b9), CLOCK.b9 (Pin_b9), CPU.b9 (Pin_b9), J10.b9 (Pin_b9), J6.b9 (Pin_b9), J7.b9 (Pin_b9), J8.b9 (Pin_b9), J9.b9 (Pin_b9)
- new net ADDR0: J1.b31 (Pin_b31)
- new net ADDR1: J1.b30 (Pin_b30)
- new net ADDR10: J1.b21 (Pin_b21)
- new net ADDR11: J1.b20 (Pin_b20)
- new net ADDR12: J1.b19 (Pin_b19)
- new net ADDR13: J1.b18 (Pin_b18)
- new net ADDR14: J1.b17 (Pin_b17)
- new net ADDR15: J1.b16 (Pin_b16)
- new net ADDR16: J1.b15 (Pin_b15)
- new net ADDR17: J1.b14 (Pin_b14)
- new net ADDR18: J1.b13 (Pin_b13)
- new net ADDR19: J1.b12 (Pin_b12)
- new net ADDR2: J1.b29 (Pin_b29)
- new net ADDR3: J1.b28 (Pin_b28)
- new net ADDR4: J1.b27 (Pin_b27)
- new net ADDR5: J1.b26 (Pin_b26)
- new net ADDR6: J1.b25 (Pin_b25)
- new net ADDR7: J1.b24 (Pin_b24)
- new net ADDR8: J1.b23 (Pin_b23)
- new net ADDR9: J1.b22 (Pin_b22)
- new net CPU/!IORD: J1.a14 (Pin_a14)
- new net CPU/!IOWR: J1.a13 (Pin_a13)
- new net CPU/5V: J1.a29 (Pin_a29), J1.a3 (Pin_a3)
- new net CPU/GND: J1.a1 (Pin_a1), J1.a10 (Pin_a10), J1.a31 (Pin_a31)
- new net CPU/READY: J1.a2 (Pin_a2)
- new net DATA0: J1.b9 (Pin_b9)
- new net DATA1: J1.b8 (Pin_b8)
- new net DATA2: J1.b7 (Pin_b7)
- new net DATA3: J1.b6 (Pin_b6)
- new net DATA4: J1.b5 (Pin_b5)
- new net DATA5: J1.b4 (Pin_b4)
- new net DATA6: J1.b3 (Pin_b3)
- new net DATA7: J1.b2 (Pin_b2)
- new net IR2: J1.a4 (Pin_a4)
- new net IR3: J1.a25 (Pin_a25)
- new net IR4: J1.a24 (Pin_a24)
- new net IR5: J1.a23 (Pin_a23)
- new net IR6: J1.a22 (Pin_a22)
- new net IR7: J1.a21 (Pin_a21)
- no-connect marks 0 -> 4
Other:
- sheet CPU ports: added !BHE, !INTA, !IORD, !IOWR, !MRD, !MWR, !TEST, 5V, ADDR[0..19], CLK, DATA[0..15], GND, HLDA, HOLD, INTR, IR[0..7], NMI, READY, RESET; removed none
- sheet Clock ports: added 5V, GND, IOCHRDY; removed none
