File: Kicad/Clock.kicad_sch (KiCad schematic)
At the start: 4 parts, among them SW1 RST, U2 8284, Y1 Crystal 30MHz

Commit message: Add files via upload
Parts:
- added R2: 10k, Resistor_THT:R_Axial_DIN0204_L3.6mm_D1.6mm_P5.08mm_Horizontal, symbol Device:R
Connections:
- net !RES: now also R1.2, U2.11 (~{RES}); no longer R1.1, U2.18 (VCC), U2.4 (RDY1)
- new net 5V: R1.1, R2.1, U2.18 (VCC)
- new net IOCHRDY: R2.2, U2.4 (RDY1)
Other:
- moved on the sheet: R1, SW1
Changed lines of the file:
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@@
 	)
 	(junction
-		(at 105.41 82.55)
+		(at 102.87 82.55)
 		(diameter 0)
 		(color 0 0 0 0)
@@
 		(color 0 0 0 0)
 	)
+	(junction
+		(at 113.03 82.55)
+		(diameter 0)
+		(color 0 0 0 0)
+	)
 	(wire
 		(pts
@@
 	(wire
 		(pts
-			(xy 95.25 118.11) (xy 111.76 118.11)
+			(xy 101.6 118.11) (xy 111.76 118.11)
 		)
 		(stroke
@@
 	(wire
 		(pts
+			(xy 110.49 82.55) (xy 113.03 82.55)
+		)
+		(stroke
+			(width 0)
+			(type default)
+		)
+	)
+	(wire
+		(pts
 			(xy 111.76 100.33) (xy 113.03 100.33)
 		)
@@
 	(wire
 		(pts
-			(xy 105.41 77.47) (xy 123.19 77.47)
-		)
-		(stroke
-			(width 0)
-			(type default)
-		)
-	)
-	(wire
-		(pts
-			(xy 105.41 87.63) (xy 105.41 82.55)
+			(xy 111.76 74.93) (xy 113.03 76.2)
+		)
+		(stroke
+			(width 0)
+			(type default)
+		)
+	)
+	(wire
+		(pts
+			(xy 113.03 76.2) (xy 113.03 82.55)
+		)
+		(stroke
+			(width 0)
+			(type default)
+		)
+	)
+	(wire
+		(pts
+			(xy 102.87 77.47) (xy 123.19 77.47)
+		)
+		(stroke
+			(width 0)
+			(type default)
+		)
+	)
+	(wire
+		(pts
+			(xy 102.87 87.63) (xy 102.87 82.55)
 		)
 		(stroke
@@
 	(wire
 		(pts
-			(xy 113.03 87.63) (xy 105.41 87.63)
+			(xy 110.49 87.63) (xy 113.03 87.63)
 		)
 		(stroke
@@
 	(wire
 		(pts
-			(xy 95.25 82.55) (xy 95.25 118.11)
+			(xy 101.6 74.93) (xy 101.6 118.11)
 		)
 		(stroke
@@
 	(wire
 		(pts
-			(xy 105.41 82.55) (xy 105.41 77.47)
+			(xy 102.87 82.55) (xy 102.87 77.47)
 		)
 		(stroke
@@
 	(hierarchical_label "5V"
 		(shape bidirectional)
-		(at 123.19 77.47 90)
+		(at 120.65 77.47 90)
 		(effects
 			(font
@@
 		)
 	)
+	(hierarchical_label "CLK"
+		(shape bidirectional)
+		(at 133.35 82.55 0)
+		(effects
+			(font
+				(size 1.27 1.27)
+			)
+			(justify left)
+		)
+	)
+	(hierarchical_label "OSC"
+		(shape bidirectional)
+		(at 133.35 100.33 0)
+		(effects
+			(font
+				(size 1.27 1.27)
+			)
+			(justify left)
+		)
+	)
 	(hierarchical_label "!RES"
 		(shape bidirectional)
-		(at 105.41 77.47 90)
-		(effects
-			(font
-				(size 1.27 1.27)
-			)
-			(justify left)
-		)
-	)
-	(hierarchical_label "CLK"
-		(shape bidirectional)
-		(at 133.35 82.55 0)
-		(effects
-			(font
-				(size 1.27 1.27)
-			)
-			(justify left)
-		)
-	)
-	(hierarchical_label "OSC"
-		(shape bidirectional)
-		(at 133.35 100.33 0)
-		(effects
-			(font
-				(size 1.27 1.27)
-			)
-			(justify left)
+		(at 113.03 82.55 270)
+		(effects
+			(font
+				(size 1.27 1.27)
+			)
+			(justify right)
 		)
 	)
@@
 		(shape bidirectional)
 		(at 123.19 118.11 270)
+		(effects
+			(font
+				(size 1.27 1.27)
+			)
+			(justify right)
+		)
+	)
+	(hierarchical_label "IOCHRDY"
+		(shape bidirectional)
+		(at 110.49 87.63 270)
 		(effects
 			(font
@@
 	(symbol
 		(lib_id "Switch:SW_Push")
-		(at 100.33 82.55 0)
+		(at 106.68 74.93 0)
 		(unit 1)
 		(body_style 1)
@@
 		(fields_autoplaced yes)
 		(property "Reference" "SW1"
-			(at 100.33 74.93 0)
+			(at 106.68 67.31 0)
 			(show_name no)
 			(do_not_autoplace no)
@@
 		)
 		(property "Value" "RST"
-			(at 100.33 77.47 0)
+			(at 106.68 69.85 0)
 			(show_name no)
 			(do_not_autoplace no)
@@
 		)
 		(property "Footprint" "Button_Switch_THT:SW_PUSH_6mm"
-			(at 100.33 77.47 0)
+			(at 106.68 69.85 0)
 			(hide yes)
 			(show_name no)
@@
 		)
 		(property "Datasheet" ""
-			(at 100.33 77.47 0)
+			(at 106.68 69.85 0)
 			(hide yes)
 			(show_name no)
@@
 		)
 		(property "Description" "Push button switch, generic, two pins"
-			(at 100.33 82.55 0)
+			(at 106.68 74.93 0)
 			(hide yes)
 			(show_name no)
@@
 	(symbol
 		(lib_id "Device:R")
-		(at 109.22 82.55 90)
+		(at 106.68 87.63 90)
+		(unit 1)
+		(body_style 1)
+		(exclude_from_sim no)
+		(in_bom yes)
+		(on_board yes)
+		(in_pos_files yes)
+		(dnp no)
+		(fields_autoplaced yes)
+		(property "Reference" "R2"
+			(at 106.68 81.28 90)
+			(show_name no)
+			(do_not_autoplace no)
+			(effects
+				(font
+					(size 1.27 1.27)
+				)
+			)
+		)
+		(property "Value" "10k"
+			(at 106.68 83.82 90)
+			(show_name no)
+			(do_not_autoplace no)
+			(effects
+				(font
+					(size 1.27 1.27)
+				)
+			)
+		)
+		(property "Footprint" "Resistor_THT:R_Axial_DIN0204_L3.6mm_D1.6mm_P5.08mm_Horizontal"
+			(at 106.68 89.408 90)
+			(hide yes)
+			(show_name no)
+			(do_not_autoplace no)
+			(effects
+				(font
+					(size 1.27 1.27)
+				)
+			)
+		)
+		(property "Datasheet" ""
+			(at 106.68 87.63 0)
+			(hide yes)
+			(show_name no)
+			(do_not_autoplace no)
+			(effects
+				(font
+					(size 1.27 1.27)
+				)
+			)
+		)
+		(property "Description" "Resistor"
+			(at 106.68 87.63 0)
+			(hide yes)
+			(show_name no)
+			(do_not_autoplace no)
+			(effects
+				(font
+					(size 1.27 1.27)
+				)
+			)
+		)
+		(pin "2"
+		)
+		(pin "1"
+		)
+		(instances
+			(project "8086testCircuit"
+				(path "/2c523d3e-2011-4584-b276-b8b67dcb79f5/a54df712-fd98-404d-b8a5-1ee8b8f9a694"
+					(reference "R2")
+					(unit 1)
+				)
+			)
+		)
+	)
+	(symbol
+		(lib_id "Device:R")
+		(at 106.68 82.55 90)
 		(unit 1)
 		(body_style 1)
@@
 		(fields_autoplaced yes)
 		(property "Reference" "R1"
-			(at 109.22 76.2 90)
+			(at 106.68 76.2 90)
 			(show_name no)
 			(do_not_autoplace no)
@@
 		)
 		(property "Value" "10k"
-			(at 109.22 78.74 90)
+			(at 106.68 78.74 90)
 			(show_name no)
 			(do_not_autoplace no)
@@
 		)
 		(property "Footprint" "Resistor_THT:R_Axial_DIN0204_L3.6mm_D1.6mm_P5.08mm_Horizontal"
-			(at 109.22 84.328 90)
+			(at 106.68 84.328 90)
 			(hide yes)
 			(show_name no)
@@
 		)
 		(property "Datasheet" ""
-			(at 109.22 82.55 0)
+			(at 106.68 82.55 0)
 			(hide yes)
 			(show_name no)
@@
 		)
 		(property "Description" "Resistor"
-			(at 109.22 82.55 0)
-			(hide yes)
-			(show_name no)
+			(at 106.68 82.55 0)
+			(hide yes)
+			(show_name no)
